File: shield-be/.history/power.kicad_sch (KiCad schematic)
At the start: 65 parts, among them J301 USB_C_Receptacle_PowerOnly_6P, J302 USB_TP, J303 JST S2B-PH-SM4-TB(LF)(SN), Q301 AO3401A, Q302 2N7002, Q303 AO3401A, Q304 SS8050, Q305 NPN, Q306 AO3401A, Q307 2N7002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

Commit message: ATDT-1.0.1
Fixes and improvements from 1.0.0 prototype
Parts:
- added D308: 1N4148, Diode_SMD:D_SOD-323, symbol Diode:1N4148
- added D309: SS14, Diode_SMD:D_SMA, symbol Diode:SS14
- added D310: 1N4148, Diode_SMD:D_SOD-323_HandSoldering, symbol Diode:1N4148
- added J304: (no value), Library:BridgePads, symbol Symbols:5mm_pad_bridge
- added R333: 0R, Resistor_SMD:R_0805_2012Metric_Pad1.20x1.40mm_HandSolder, symbol 2-altium-import:root_3_CMP-1853144-2_CommunityVault_0
- R305: value 100k -> 10k; LCSC C149504 -> C17414
- R322: now left out of the parts list
Connections:
- net BATT_P: now also D309.2 (A); no longer R305.1
- net GND: now also R303.2
- net PWR_VIN: now also D309.1 (K); no longer R303.2
- net PWR_VOUT: now also R305.2
- net USB_P: now also D308.2 (A)
- net at D305.1 (K), D306.1 (K), Q305.2 (C)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: now also J304.2 (B), R333.1
- net at Q301.1 (G), R303.1: now also D308.1 (K); no longer R305.2
- new net: D310.2 (A), R305.1
- new net: D310.1 (K), J304.1 (A), R333.2
Other:
- note added: "-=BATTERY/USB POWER SELECTION=- Just use a diode to prevent backfeed over USB, power waste here isn't an issue. Use a enhancment P-Fet as an ideal diode that lets current flow when PWR_VIN is lower than BATT_P. (Extra diode to deal with some transient situations where the fet is slightly too slow to respond) No protection for LIPO over-discharge. (Use battery with BMS)"
- note added: "Optional bridge to disable soft-off. (Useful for flashing initial firmware) Populate R333 to make permenant"
- note removed: "-=BATTERY/USB POWER SELECTION=- Just use a diode to prevent backfeed over USB, power waste here isn't an issue. Use a enhancment P-Fet as an ideal diode that lets current flow when PWR_VIN is lower than BATT_P No protection for LIPO over-discharge. (Use battery with BMS)"
- moved on the sheet: C301, C302, C303, R303, R330
